File: electrical/dif-pressure-meter.kicad_pcb (KiCad board)
At the start: 2 copper layers, 41 x 87 mm, 68 parts, among them J1 USB_C_Receptacle_USB2.0, J2 JST PH2, J3 Conn_01x06, J4 Conn_01x07, J5 Conn_01x04, Q1 SIL2308-TP, Q2 BC817, Q3 BC817, Q4 SIL2308-TP, Q5 SIL2308-TP, Q6 BC817, SW1 SWITCH_5WAY_8x8, U1 CH340C, U2 TP4056, U3 RT9080-33GJ5, U4 ESP32-WROOM-E, U5 LCD_ST7735S_1.8

Commit message: electrical fixes v1.1
Routing:
- net /PWR_SW: track 78.3 -> 71.9 mm
- net /GPIO19: track 67.0 -> 71.9 mm, vias 1 -> 2
- net /GPIO17: track 60.4 -> 63.4 mm
- net /GPIO33: track 68.2 -> 71.2 mm
- net /GPIO32: track 80.0 -> 83.0 mm
- net /KEYS_BL: track 51.8 -> 54.4 mm
- net Net-(SW1-LED_L): track 42.6 -> 40.4 mm
- net Net-(SW1-LED_R): track 12.2 -> 13.7 mm
- net Net-(SW1-LED_C): track 18.2 -> 18.9 mm
- net GND: vias 58 -> 60
Other:
- board text added: "v1.1"
- board text removed: "v1.0"

Commit message: updated schematic
Parts:
- D3: value 1N5819HW-7-F -> 1N4148W; footprint footprints:SOD3715X145N -> Diode_SMD:D_SOD-123F
- R23, R24: value 2.2 -> 2.2k
- moved D3 0.10 mm to (137.9, 62.5)
Routing:
- net /PWR_SW: track 71.9 -> 72.4 mm
Changed lines of the file:
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@@
       (net 42 "/SCREEN_BL") (pinfunction "BL") (pintype "input"))
     (model "${KIPRJMOD}/3dmodels/1.8_lcd.step"
-      (offset (xyz 1 23.9 4))
+      (offset (xyz 1 23.9 4.2))
       (scale (xyz 1 1 1))
       (rotate (xyz 0 180 180))
@@
       )
     )
+    (model "${KIPRJMOD}/3dmodels/5way-switch.step"
+      (offset (xyz 0 0 5.5))
+      (scale (xyz 1 1 1))
+      (rotate (xyz 0 0 0))
+    )
   )
   (footprint "Resistor_SMD:R_0805_2012Metric_Pad1.20x1.40mm_HandSolder" (layer "B.Cu")
@@
     )
   )
-  (footprint "footprints:SOD3715X145N" (layer "B.Cu")
-    (at 138 62.5 90)
+  (footprint "Diode_SMD:D_SOD-123F" (layer "B.Cu")
+    (at 137.9 62.5 90)
+    (descr "D_SOD-123F")
+    (tags "D_SOD-123F")
     (property "Availability" "In Stock")
     (property "Check_prices" "https://www.snapeda.com/parts/1N5819HW-7-F/Diodes+Inc./view-part/?ref=eda")
@@
     (property "Sheetfile" "dif-pressure-meter.kicad_sch")
     (property "Sheetname" "")
+    (property "Sim.Device" "D")
+    (property "Sim.Pins" "1=K 2=A")
     (property "SnapEDA_Link" "https://www.snapeda.com/parts/1N5819HW-7-F/Diodes+Inc./view-part/?ref=snap")
+    (property "ki_description" "75V 0.15A Fast Switching Diode, SOD-123")
+    (property "ki_keywords" "diode")
     (attr smd)
-    (fp_text reference "D3" (at 0 -1.7 270) (layer "B.SilkS")
-        (effects (font (size 0.8 0.8) (thickness 0.15)) (justify mirror))
+    (fp_text reference "D3" (at 0 -1.8 270) (layer "B.SilkS")
+        (effects (font (size 1 1) (thickness 0.15)) (justify mirror))
     )
-    (fp_text value "1N5819HW-7-F" (at 1.158204 -1.445961 270) (layer "B.Fab")
-        (effects (font (size 0.8 0.8) (thickness 0.15)) (justify mirror))
+    (fp_text value "1N4148W" (at 0 -2.1 270) (layer "B.Fab")
+        (effects (font (size 1 1) (thickness 0.15)) (justify mirror))
     )
-    (fp_line (start -1.425 0.85) (end 1.425 0.85)
-      (stroke (width 0.127) (type solid)) (layer "B.SilkS"))
-    (fp_line (start 1.425 -0.85) (end -1.425 -0.85)
-      (stroke (width 0.127) (type solid)) (layer "B.SilkS"))
-    (fp_circle (center -3 0) (end -2.9 0)
-      (stroke (width 0.2) (type solid)) (fill none) (layer "B.SilkS"))
-    (fp_line (start -2.535 -1.1) (end -2.535 1.1)
+    (fp_text user "${REFERENCE}" (at -0.127 1.905 270) (layer "B.Fab")
+        (effects (font (size 1 1) (thickness 0.15)) (justify mirror))
+    )
+    (fp_line (start -2.21 -1) (end 1.65 -1)
+      (stroke (width 0.12) (type solid)) (layer "B.SilkS"))
+    (fp_line (start -2.21 1) (end -2.21 -1)
+      (stroke (width 0.12) (type solid)) (layer "B.SilkS"))
+    (fp_line (start -2.21 1) (end 1.65 1)
+      (stroke (width 0.12) (type solid)) (layer "B.SilkS"))
+    (fp_line (start -2.2 1.15) (end -2.2 -1.15)
       (stroke (width 0.05) (type solid)) (layer "B.CrtYd"))
-    (fp_line (start -2.535 1.1) (end 2.535 1.1)
+    (fp_line (start -2.2 1.15) (end 2.2 1.15)
       (stroke (width 0.05) (type solid)) (layer "B.CrtYd"))
-    (fp_line (start 2.535 -1.1) (end -2.535 -1.1)
+    (fp_line (start 2.2 -1.15) (end -2.2 -1.15)
       (stroke (width 0.05) (type solid)) (layer "B.CrtYd"))
-    (fp_line (start 2.535 1.1) (end 2.535 -1.1)
+    (fp_line (start 2.2 1.15) (end 2.2 -1.15)
       (stroke (width 0.05) (type solid)) (layer "B.CrtYd"))
-    (fp_line (start -1.425 -0.85) (end -1.425 0.85)
-      (stroke (width 0.127) (type solid)) (layer "B.Fab"))
-    (fp_line (start -1.425 0.85) (end 1.425 0.85)
-      (stroke (width 0.127) (type solid)) (layer "B.Fab"))
-    (fp_line (start 1.425 -0.85) (end -1.425 -0.85)
-      (stroke (width 0.127) (type solid)) (layer "B.Fab"))
-    (fp_line (start 1.425 0.85) (end 1.425 -0.85)
-      (stroke (width 0.127) (type solid)) (layer "B.Fab"))
-    (fp_circle (center -3 0) (end -2.9 0)
-      (stroke (width 0.2) (type solid)) (fill none) (layer "B.Fab"))
-    (pad "A" smd rect (at 1.68 0 90) (size 1.21 0.73) (layers "B.Cu" "B.Paste" "B.Mask")
-      (net 38 "/GPIO16") (pintype "passive") (solder_mask_margin 0.102))
-    (pad "C" smd rect (at -1.68 0 90) (size 1.21 0.73) (layers "B.Cu" "B.Paste" "B.Mask")
-      (net 35 "/PWR_SW") (pintype "passive") (solder_mask_margin 0.102))
-    (model ":KICAD7_3DMODEL_DIR:Diode_SMD.3dshapes/D_SOD-123F.step"
+    (fp_line (start -1.4 -0.9) (end -1.4 0.9)
+      (stroke (width 0.1) (type solid)) (layer "B.Fab"))
+    (fp_line (start -1.4 0.9) (end 1.4 0.9)
+      (stroke (width 0.1) (type solid)) (layer "B.Fab"))
+    (fp_line (start -0.75 0) (end -0.35 0)
+      (stroke (width 0.1) (type solid)) (layer "B.Fab"))
+    (fp_line (start -0.35 0) (end -0.35 -0.55)
+      (stroke (width 0.1) (type solid)) (layer "B.Fab"))
+    (fp_line (start -0.35 0) (end -0.35 0.55)
+      (stroke (width 0.1) (type solid)) (layer "B.Fab"))
+    (fp_line (start -0.35 0) (end 0.25 0.4)
+      (stroke (width 0.1) (type solid)) (layer "B.Fab"))
+    (fp_line (start 0.25 -0.4) (end -0.35 0)
+      (stroke (width 0.1) (type solid)) (layer "B.Fab"))
+    (fp_line (start 0.25 0) (end 0.75 0)
+      (stroke (width 0.1) (type solid)) (layer "B.Fab"))
+    (fp_line (start 0.25 0.4) (end 0.25 -0.4)
+      (stroke (width 0.1) (type solid)) (layer "B.Fab"))
+    (fp_line (start 1.4 -0.9) (end -1.4 -0.9)
+      (stroke (width 0.1) (type solid)) (layer "B.Fab"))
+    (fp_line (start 1.4 0.9) (end 1.4 -0.9)
+      (stroke (width 0.1) (type solid)) (layer "B.Fab"))
+    (pad "1" smd roundrect (at -1.4 0 90) (size 1.1 1.1) (layers "B.Cu" "B.Paste" "B.Mask") (roundrect_rratio 0.2272727273)
+      (net 35 "/PWR_SW") (pinfunction "K") (pintype "passive"))
+    (pad "2" smd roundrect (at 1.4 0 90) (size 1.1 1.1) (layers "B.Cu" "B.Paste" "B.Mask") (roundrect_rratio 0.2272727273)
+      (net 38 "/GPIO16") (pinfunction "A") (pintype "passive"))
+    (model "${KICAD6_3DMODEL_DIR}/Diode_SMD.3dshapes/D_SOD-123F.wrl"
       (offset (xyz 0 0 0))
       (scale (xyz 1 1 1))
@@
         (effects (font (size 0.8 0.8) (thickness 0.15)) (justify mirror))
     )
-    (fp_text value "2.2" (at 0 -1.65) (layer "B.Fab")
+    (fp_text value "2.2k" (at 0 -1.65) (layer "B.Fab")
         (effects (font (size 0.8 0.8) (thickness 0.15)) (justify mirror))
     )
@@
         (effects (font (size 0.8 0.8) (thickness 0.15)) (justify mirror))
     )
-    (fp_text value "2.2" (at 0 -1.65) (layer "B.Fab")
+    (fp_text value "2.2k" (at 0 -1.65) (layer "B.Fab")
         (effects (font (size 0.8 0.8) (thickness 0.15)) (justify mirror))
     )
@@
   (via (at 146.1 77.2) (size 0.8) (drill 0.4) (layers "F.Cu" "B.Cu") (free) (net 12))
   (via (at 111.6 120.1) (size 0.8) (drill 0.4) (layers "F.Cu" "B.Cu") (free) (net 12))
-  (via (at 136.4 60.1) (size 0.8) (drill 0.4) (layers "F.Cu" "B.Cu") (free) (net 12))
+  (via (at 136.2 59.7) (size 0.8) (drill 0.4) (layers "F.Cu" "B.Cu") (free) (net 12))
   (via (at 139.9 107.5) (size 0.8) (drill 0.4) (layers "F.Cu" "B.Cu") (free) (net 12))
   (via (at 134 102.1) (size 0.8) (drill 0.4) (layers "F.Cu" "B.Cu") (free) (net 12))
@@
   (via (at 139.125 65.875) (size 0.8) (drill 0.4) (layers "F.Cu" "B.Cu") (net 35))
   (segment (start 139.9625 64.4625) (end 140 64.5) (width 0.4) (layer "B.Cu") (net 35))
-  (segment (start 139.68 64.18) (end 140 64.5) (width 0.4) (layer "B.Cu") (net 35))
-  (segment (start 139.125 65.875) (end 138 64.75) (width 0.4) (layer "B.Cu") (net 35))
+  (segment (start 139.4 63.9) (end 140 64.5) (width 0.4) (layer "B.Cu") (net 35))
+  (segment (start 137.9 64.65) (end 137.9 63.9) (width 0.4) (layer "B.Cu") (net 35))
+  (segment (start 137.9 63.9) (end 139.4 63.9) (width 0.4) (layer "B.Cu") (net 35))
   (segment (start 139.9625 62.25) (end 139.9625 64.4625) (width 0.4) (layer "B.Cu") (net 35))
-  (segment (start 138 64.18) (end 139.68 64.18) (width 0.4) (layer "B.Cu") (net 35))
-  (segment (start 138 64.75) (end 138 64.18) (width 0.4) (layer "B.Cu") (net 35))
+  (segment (start 139.125 65.875) (end 137.9 64.65) (width 0.4) (layer "B.Cu") (net 35))
   (segment (start 138.5495 52.75) (end 143.5 52.75) (width 0.4) (layer "F.Cu") (net 36))
   (via (at 138.5495 52.75) (size 0.8) (drill 0.4) (layers "F.Cu" "B.Cu") (net 36))
@@
   (via (at 132.260332 62.739668) (size 0.8) (drill 0.4) (layers "F.Cu" "B.Cu") (net 38))
   (via (at 139.058557 56.641917) (size 0.8) (drill 0.4) (layers "F.Cu" "B.Cu") (net 38))
+  (segment (start 136.25 62.75) (end 138 61) (width 0.4) (layer "B.Cu") (net 38))
   (segment (start 143 48) (end 144.45 48) (width 0.4) (layer "B.Cu") (net 38))
   (segment (start 139.058557 56.641917) (end 138 57.700474) (width 0.4) (layer "B.Cu") (net 38))
-  (segment (start 138 58.43) (end 138 60.82) (width 0.4) (layer "B.Cu") (net 38))
+  (segment (start 132.270664 62.75) (end 136.25 62.75) (width 0.4) (layer "B.Cu") (net 38))
   (segment (start 141 47.75) (end 142.75 47.75) (width 0.4) (layer "B.Cu") (net 38))
+  (segment (start 138 61) (end 138 58.43) (width 0.4) (layer "B.Cu") (net 38))
   (segment (start 130.5 64.47) (end 130.47 64.5) (width 0.4) (layer "B.Cu") (net 38))
-  (segment (start 132.260332 62.739668) (end 132.270664 62.75) (width 0.4) (layer "B.Cu") (net 38))
   (segment (start 142.75 47.75) (end 143 48) (width 0.4) (layer "B.Cu") (net 38))
   (segment (start 130.5 63.25) (end 130.5 64.47) (width 0.4) (layer "B.Cu") (net 38))
-  (segment (start 132.270664 62.75) (end 136.07 62.75) (width 0.4) (layer "B.Cu") (net 38))
-  (segment (start 136.07 62.75) (end 138 60.82) (width 0.4) (layer "B.Cu") (net 38))
+  (segment (start 132.260332 62.739668) (end 132.270664 62.75) (width 0.4) (layer "B.Cu") (net 38))
   (segment (start 138 57.700474) (end 138 58.43) (width 0.4) (layer "B.Cu") (net 38))
   (segment (start 144.45 48) (end 147.75 51.3) (width 0.4) (layer "B.Cu") (net 38))
