File: electrical/dif-pressure-meter.kicad_sch (KiCad schematic)
At the start: 68 parts, among them J1 USB_C_Receptacle_USB2.0, J2 JST PH2, J3 Conn_01x06, J4 Conn_01x07, J5 Conn_01x04, Q1 SIL2308-TP, Q2 BC817, Q3 BC817, Q4 SIL2308-TP, Q5 SIL2308-TP, Q6 BC817, SW1 SWITCH_5WAY_8x8, U1 CH340C, U2 TP4056, U3 RT9080-33GJ5, U4 ESP32-WROOM-E, U5 LCD_ST7735S_1.8

Commit message: electrical fixes v1.1
Parts:
- R23, R24: value 2.2 -> 2.2k
Other:
- note added: "1.3mA per LED"
Changed lines of the file:
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@@
     (title "Differential pressure meter")
     (date "2023-10-06")
-    (rev "1.0")
+    (rev "1.1")
   )
   (junction (at 66.04 46.99) (diameter 0) (color 0 0 0 0)
@@
   (text "Battery charger:" (at 15.24 153.67 0)
     (effects (font (size 1.27 1.27) (thickness 0.254) bold) (justify left bottom))
+  )
+  (text "1.3mA per LED" (at 355.6 57.15 0)
+    (effects (font (size 1.27 1.27)) (justify left bottom))
   )
   (label "GPIO26" (at 347.98 71.12 0) (fields_autoplaced)
@@
       (effects (font (size 1.27 1.27)) (justify left))
     )
-    (property "Value" "2.2" (at 361.95 171.45 0)
+    (property "Value" "2.2k" (at 361.95 171.45 0)
       (effects (font (size 1.27 1.27)) (justify left))
     )
@@
       (effects (font (size 1.27 1.27)) (justify left))
     )
-    (property "Value" "2.2" (at 361.95 191.77 0)
+    (property "Value" "2.2k" (at 361.95 191.77 0)
       (effects (font (size 1.27 1.27)) (justify left))
     )

Commit message: updated schematic
Parts:
- D3: value 1N5819HW-7-F -> 1N4148W; footprint footprints:SOD3715X145N -> Diode_SMD:D_SOD-123F; symbol 1N5819HW-7-F:1N5819HW-7-F -> Diode:1N4148W
Connections:
- net GPIO16: now also D3.2 (A); no longer D3.A
- net PWR_SW: now also D3.1 (K); no longer D3.C
Other:
- note added: "Based on: https://www.sparkfun.com/products/17870"
- note added: "Measured power-off current draw: 11.7 uA"
- note added: "fast off"
- note added: "power sense"
Changed lines of the file:
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@@
     (stroke (width 0) (type default))
   )
-  (wire (pts (xy 104.14 66.04) (xy 104.14 62.23))
+  (wire (pts (xy 104.14 62.23) (xy 104.14 66.04))
     (stroke (width 0) (type default))
   )
@@
     (stroke (width 0) (type default))
   )
-  (wire (pts (xy 104.14 49.53) (xy 104.14 52.07))
+  (wire (pts (xy 104.14 49.53) (xy 104.14 54.61))
     (stroke (width 0) (type default))
   )
@@
     (effects (font (size 1.27 1.27) (thickness 0.254) bold) (justify left bottom))
   )
+  (text "Based on: https://www.sparkfun.com/products/17870" (at 123.19 104.14 0)
+    (effects (font (size 1.27 1.27)) (justify left bottom))
+  )
   (text "Sensor:" (at 336.55 153.67 0)
     (effects (font (size 1.27 1.27) (thickness 0.254) bold) (justify left bottom))
@@
     (effects (font (size 1.27 1.27) (thickness 0.254) bold) (justify left bottom))
   )
+  (text "fast off" (at 161.29 54.61 0)
+    (effects (font (size 1.27 1.27)) (justify left bottom))
+  )
+  (text "power sense" (at 161.29 64.77 0)
+    (effects (font (size 1.27 1.27)) (justify left bottom))
+  )
   (text "ESP32:" (at 181.61 29.21 0)
     (effects (font (size 1.27 1.27) (thickness 0.254) bold) (justify left bottom))
@@
   )
   (text "1.3mA per LED" (at 355.6 57.15 0)
+    (effects (font (size 1.27 1.27)) (justify left bottom))
+  )
+  (text "Measured power-off current draw: 11.7 uA" (at 26.67 271.78 0)
     (effects (font (size 1.27 1.27)) (justify left bottom))
   )
@@
     )
   )
-  (symbol (lib_id "1N5819HW-7-F:1N5819HW-7-F") (at 104.14 57.15 90) (unit 1)
+  (symbol (lib_id "Diode:1N4148W") (at 104.14 58.42 270) (unit 1)
     (in_bom yes) (on_board yes) (dnp no) (fields_autoplaced)
-    (property "Reference" "D3" (at 106.68 55.88 90)
-      (effects (font (size 1.27 1.27)) (justify right))
-    )
-    (property "Value" "1N5819HW-7-F" (at 106.68 58.42 90)
-      (effects (font (size 1.27 1.27)) (justify right))
-    )
-    (property "Footprint" "footprints:SOD3715X145N" (at 104.14 57.15 0)
-      (effects (font (size 1.27 1.27)) (justify bottom) hide)
-    )
-    (property "Datasheet" "" (at 104.14 57.15 0)
-      (effects (font (size 1.27 1.27)) hide)
-    )
-    (property "MF" "Diodes Inc." (at 104.14 57.15 0)
-      (effects (font (size 1.27 1.27)) (justify bottom) hide)
-    )
-    (property "Description" "\nDiode Schottky 1A 40V SOD123 | Diodes Inc 1N5819HW-7-F\n" (at 104.14 57.15 0)
-      (effects (font (size 1.27 1.27)) (justify bottom) hide)
-    )
-    (property "Package" "SOD-123 Fairchild Semiconductor" (at 104.14 57.15 0)
-      (effects (font (size 1.27 1.27)) (justify bottom) hide)
-    )
-    (property "Price" "None" (at 104.14 57.15 0)
-      (effects (font (size 1.27 1.27)) (justify bottom) hide)
-    )
-    (property "Check_prices" "https://www.snapeda.com/parts/1N5819HW-7-F/Diodes+Inc./view-part/?ref=eda" (at 104.14 57.15 0)
-      (effects (font (size 1.27 1.27)) (justify bottom) hide)
-    )
-    (property "STANDARD" "IPC-7351B" (at 104.14 57.15 0)
-      (effects (font (size 1.27 1.27)) (justify bottom) hide)
-    )
-    (property "PARTREV" "18-2" (at 104.14 57.15 0)
-      (effects (font (size 1.27 1.27)) (justify bottom) hide)
-    )
-    (property "SnapEDA_Link" "https://www.snapeda.com/parts/1N5819HW-7-F/Diodes+Inc./view-part/?ref=snap" (at 104.14 57.15 0)
-      (effects (font (size 1.27 1.27)) (justify bottom) hide)
-    )
-    (property "MP" "1N5819HW-7-F" (at 104.14 57.15 0)
-      (effects (font (size 1.27 1.27)) (justify bottom) hide)
-    )
-    (property "Purchase-URL" "https://www.snapeda.com/api/url_track_click_mouser/?unipart_id=42272&manufacturer=Diodes Inc.&part_name=1N5819HW-7-F&search_term=None" (at 104.14 57.15 0)
-      (effects (font (size 1.27 1.27)) (justify bottom) hide)
-    )
-    (property "Availability" "In Stock" (at 104.14 57.15 0)
-      (effects (font (size 1.27 1.27)) (justify bottom) hide)
-    )
-    (property "MANUFACTURER" "Diodes Inc." (at 104.14 57.15 0)
-      (effects (font (size 1.27 1.27)) (justify bottom) hide)
-    )
-    (pin "A")
-    (pin "C")
-    (instances
-      (project "dif-pressure-meter"
+    (property "Reference" "D3" (at 106.68 57.15 90)
+      (effects (font (size 1.27 1.27)) (justify left))
+    )
+    (property "Value" "1N4148W" (at 106.68 59.69 90)
+      (effects (font (size 1.27 1.27)) (justify left))
+    )
+    (property "Footprint" "Diode_SMD:D_SOD-123F" (at 99.695 58.42 0)
+      (effects (font (size 1.27 1.27)) hide)
+    )
+    (property "Datasheet" "https://www.vishay.com/docs/85748/1n4148w.pdf" (at 104.14 58.42 0)
+      (effects (font (size 1.27 1.27)) hide)
+    )
+    (property "MF" "Diodes Inc." (at 104.14 58.42 0)
+      (effects (font (size 1.27 1.27)) (justify bottom) hide)
+    )
+    (property "Description" "\nDiode Schottky 1A 40V SOD123 | Diodes Inc 1N5819HW-7-F\n" (at 104.14 58.42 0)
+      (effects (font (size 1.27 1.27)) (justify bottom) hide)
+    )
+    (property "Package" "SOD-123 Fairchild Semiconductor" (at 104.14 58.42 0)
+      (effects (font (size 1.27 1.27)) (justify bottom) hide)
+    )
+    (property "Price" "None" (at 104.14 58.42 0)
+      (effects (font (size 1.27 1.27)) (justify bottom) hide)
+    )
+    (property "Check_prices" "https://www.snapeda.com/parts/1N5819HW-7-F/Diodes+Inc./view-part/?ref=eda" (at 104.14 58.42 0)
+      (effects (font (size 1.27 1.27)) (justify bottom) hide)
+    )
+    (property "STANDARD" "IPC-7351B" (at 104.14 58.42 0)
+      (effects (font (size 1.27 1.27)) (justify bottom) hide)
+    )
+    (property "PARTREV" "18-2" (at 104.14 58.42 0)
+      (effects (font (size 1.27 1.27)) (justify bottom) hide)
+    )
+    (property "SnapEDA_Link" "https://www.snapeda.com/parts/1N5819HW-7-F/Diodes+Inc./view-part/?ref=snap" (at 104.14 58.42 0)
+      (effects (font (size 1.27 1.27)) (justify bottom) hide)
+    )
+    (property "MP" "1N5819HW-7-F" (at 104.14 58.42 0)
+      (effects (font (size 1.27 1.27)) (justify bottom) hide)
+    )
+    (property "Purchase-URL" "https://www.snapeda.com/api/url_track_click_mouser/?unipart_id=42272&manufacturer=Diodes Inc.&part_name=1N5819HW-7-F&search_term=None" (at 104.14 58.42 0)
+      (effects (font (size 1.27 1.27)) (justify bottom) hide)
+    )
+    (property "Availability" "In Stock" (at 104.14 58.42 0)
+      (effects (font (size 1.27 1.27)) (justify bottom) hide)
+    )
+    (property "MANUFACTURER" "Diodes Inc." (at 104.14 58.42 0)
+      (effects (font (size 1.27 1.27)) (justify bottom) hide)
+    )
+    (property "Sim.Device" "D" (at 104.14 58.42 0)
+      (effects (font (size 1.27 1.27)) hide)
+    )
+    (property "Sim.Pins" "1=K 2=A" (at 104.14 58.42 0)
+      (effects (font (size 1.27 1.27)) hide)
+    )
+    (pin "1")
+    (pin "2")
+    (instances
+      (project "dif-pressure-meter"
